Commit message: fix tom link issues

File: tom_description/robots/tom_lacquey.urdf.xacro (robot description, xacro)
@@ -92,5 +92,5 @@
          <color rgba="0.92 0.63 0.08 1.0"/>
        </material>
-    </visual>
+     </visual>
   </link>
 	<joint name="box_tom_joint" type="fixed">

File: tom_description/robots/tom_table.urdf.xacro (robot description, xacro)
@@ -78,5 +78,5 @@
          <color rgba="0.00 0.25 1.0 1.0"/>
        </material>
-    </visual>
+     </visual>
   </link>
   <link name="box_tom_link">
